File: ICE40-IO_Rev_A.kicad_pcb (KiCad board)
At the start: 2 copper layers, 45 x 50 mm, 43 parts

Commit message: update
Connections:
- net /LED1 renamed /IrDA_SC
- net /LED2 renamed /IrDA_Rx
- net /PIO2_1 renamed /VGA_GREEN2
- net /PIO2_2 renamed /VGA_GREEN3
- net /PIO2_3 renamed /VGA_BLUE1
- net /PIO2_4 renamed /VGA_BLUE2
- net /PIO2_5 renamed /VGA_BLUE3
- net /PIO2_6 renamed /VGA_HSYNC
- net /PIO2_7 renamed /VGA_VSYNC
- net /PIO2_8/TxD renamed /PS2_DATA
- net /PIO2_9/RxD renamed /PS2_CLK
- net /PIO3_10A renamed /GPIO_Pin<31>
- net /PIO3_10B renamed /IrDA_Tx
- net /PIO3_12A renamed /VGA_RED3
- net /PIO3_12B renamed /VGA_GREEN1
- net /PIO3_1A renamed /GPIO_Pin<5>
- net /PIO3_1B renamed /GPIO_Pin<7>
- net /PIO3_2A renamed /GPIO_Pin<9>
- net /PIO3_2B renamed /GPIO_Pin<11>
- net /PIO3_3A renamed /GPIO_Pin<13>
- net /PIO3_3B renamed /GPIO_Pin<15>
- net /PIO3_5A renamed /GPIO_Pin<17>
- net /PIO3_5B renamed /GPIO_Pin<19>
- net /PIO3_6A renamed /GPIO_Pin<21>
- net /PIO3_6B renamed /GPIO_Pin<23>
- net /PIO3_7B renamed /GPIO_Pin<25>
- net /PIO3_8A renamed /VGA_RED1
- net /PIO3_8B renamed /VGA_RED2
