File: ICE40-IO_Rev_A.sch (KiCad schematic (older format))
At the start: 33 parts

Commit message: update
Connections:
- net labels added: GPIO_Pin<11>, GPIO_Pin<13>, GPIO_Pin<15>, GPIO_Pin<17>, GPIO_Pin<19>, GPIO_Pin<21>, GPIO_Pin<23>, GPIO_Pin<25>, GPIO_Pin<31>, GPIO_Pin<5>, GPIO_Pin<7>, GPIO_Pin<9>, IrDA_Rx, IrDA_SC, IrDA_Tx, PS2_CLK, PS2_DATA, VGA_BLUE1, VGA_BLUE2, VGA_BLUE3, VGA_GREEN1, VGA_GREEN2, VGA_GREEN3, VGA_HSYNC, VGA_RED1, VGA_RED2, VGA_RED3, VGA_VSYNC
- net labels removed: LED1, LED2, PIO2_1, PIO2_2, PIO2_3, PIO2_4, PIO2_5, PIO2_6, PIO2_7, PIO2_8/TxD, PIO2_9/RxD, PIO3_10A, PIO3_10B, PIO3_12A, PIO3_12B, PIO3_1A, PIO3_1B, PIO3_2A, PIO3_2B, PIO3_3A, PIO3_3B, PIO3_5A, PIO3_5B, PIO3_6A, PIO3_6B, PIO3_7B, PIO3_8A, PIO3_8B
